File: EngReab/Muleta/Muleta.sch (EAGLE design)
At the start: 16 parts, among them IC1 REF01Z, IC2 INA110KP, IC3 LF356N, J1 RJ11-6X

Commit message: Saida Analog A5?
Parts:
- added HC05: (no value), pinhead:PINHD-1X6/90
- added IOL1, POWER1: (no value), pinhead:PINHD-1X8
- added JP1: (no value), pinhead:PINHD-1X3
- added R10: 2k2R, resistor:R-EU_0207/7
- added R9: 1k5R, resistor:R-EU_0207/7
- C2, C3: device capacitor-wima:C2,5-3 -> capacitor-wima:C5/2.5
- C4: device capacitor-wima:C7.5/3 -> capacitor-wima:C5/2.5
Connections:
- removed net VCC: C1.1, C2.1, C3.2, IC1.V+, IC3.V+, IC3.V-, R7.1
- new net +15V: C1.1, C2.1, IC1.V+, IC2P.+VCC, IC3.V-, JP1.1, R7.1
- new net -15V: C3.2, IC2P.-VCC, IC3.V+, JP1.3
- new net ARDUINO_5V: HC05.2, POWER1.5
- new net ARDUINO_DIG: IOL1.2, R9.1
- new net ARDUINO_GND: HC05.3, POWER1.6, R10.1
- new net N$15: HC05.5, R10.2, R9.2
- net GND: now also JP1.2
Other:
- moved on the sheet: C2, C3, C4, IC2, IC3, J1, R1, R2, R3, R4, R5, R6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
